Commit message: plenty of testing in progress, but launch is stable without slam here; adding slam next

File: turtlebot3_manipulation_gazebo/urdf/turtlebot3_pi_base.xacro (robot description, xacro)
@@ -86,5 +86,7 @@
     <origin xyz="0.0 0.144 0.023" rpy="-1.57 0 0"/>
     <axis xyz="0 0 1"/>
-    <dynamics damping="0.2" friction="0.5"/>
+    <xacro:if value="$(arg gazebo)">
+      <dynamics damping="0.2" friction="0.5"/>
+    </xacro:if>
   </joint>
   <link name="wheel_right_link">
@@ -141,5 +143,7 @@
     <origin xyz="0.0 -0.144 0.023" rpy="-1.57 0 0"/>
     <axis xyz="0 0 1"/>
-    <dynamics damping="0.2" friction="0.5"/>
+    <xacro:if value="$(arg gazebo)">
+      <dynamics damping="0.2" friction="0.5"/>
+    </xacro:if>
   </joint>
   <link name="caster_back_right_link">
@@ -218,5 +222,5 @@
       <origin xyz="0 0 0" rpy="0 0 0"/>
       <axis xyz="0 0 1"/>
-      <dynamics damping="0.1" friction="0.2"/>
+     <dynamics damping="0.1" friction="0.2"/>
     </joint>
   </xacro:if>

File: turtlebot3_manipulation_gazebo/urdf/turtlebot3_pi_gazebo.xacro (robot description, xacro)
@@ -164,4 +164,40 @@
       </sensor>
     </gazebo>
+    <gazebo>
+      <plugin filename="libgazebo_ros_diff_drive.so" name="turtlebot3_diff_drive">
+        <ros>
+          <!-- <namespace>/tb3</namespace> -->
+        </ros>
+        <update_rate>30</update_rate>
+        <!-- wheels -->
+        <left_joint>wheel_left_joint</left_joint>
+        <right_joint>wheel_right_joint</right_joint>
+        <!-- kinematics -->
+        <wheel_separation>0.287</wheel_separation>
+        <wheel_diameter>0.066</wheel_diameter>
+        <!-- limits -->
+        <max_wheel_torque>20</max_wheel_torque>
+        <max_wheel_acceleration>1.0</max_wheel_acceleration>
+        <command_topic>cmd_vel</command_topic>
+        <!-- output -->
+        <publish_odom>true</publish_odom>
+        <publish_odom_tf>true</publish_odom_tf>
+        <publish_wheel_tf>false</publish_wheel_tf>
+        <odometry_topic>odom</odometry_topic>
+        <odometry_frame>odom</odometry_frame>
+        <robot_base_frame>base_footprint</robot_base_frame>
+      </plugin>
+    </gazebo>
+    <gazebo>
+      <plugin filename="libgazebo_ros_joint_state_publisher.so" name="turtlebot3_joint_state">
+        <ros>
+          <!-- <namespace>/tb3</namespace> -->
+          <remapping>~/out:=joint_states</remapping>
+        </ros>
+        <update_rate>30</update_rate>
+        <joint_name>wheel_left_joint</joint_name>
+        <joint_name>wheel_right_joint</joint_name>
+      </plugin>
+    </gazebo>
   </xacro:if>
 </robot>

File: turtlebot3_manipulation_gazebo/urdf/turtlebot3_pi_manipulator.xacro (robot description, xacro)
@@ -5,13 +5,17 @@
   <!--  TURTLEBOT3 WAFFLE PI  -->
   <xacro:include filename="$(find turtlebot3_manipulation_gazebo)/urdf/turtlebot3_pi.xacro"/>
-  <!-- OPEN MANIPULATOR X -->
-  <xacro:include filename="$(find open_manipulator_x_description)/urdf/open_manipulator_x.urdf.xacro"/>
-  <xacro:include filename="$(find open_manipulator_x_description)/urdf/open_manipulator_x.transmission.xacro"/>
-  <xacro:include filename="$(find open_manipulator_x_description)/urdf/open_manipulator_x.gazebo.xacro"/>
-  <!-- TURTLEBOT-OPEN MANIPULATOR JOINT  -->
-  <joint name="base_to_link1" type="fixed">
-    <origin xyz="-0.092 0.0 0.091" rpy="0 0 0"/>
-    <parent link="base_link"/>
-    <child link="link1"/>
-  </joint>
+  <!--  if gazebo=True, enable SDF specific tags  -->
+  <xacro:arg name="include_manipulator" default="True"/>
+  <xacro:if value="$(arg include_manipulator)">
+    <!-- OPEN MANIPULATOR X -->
+    <xacro:include filename="$(find open_manipulator_x_description)/urdf/open_manipulator_x.urdf.xacro"/>
+    <xacro:include filename="$(find open_manipulator_x_description)/urdf/open_manipulator_x.transmission.xacro"/>
+    <xacro:include filename="$(find open_manipulator_x_description)/urdf/open_manipulator_x.gazebo.xacro"/>
+    <!-- TURTLEBOT-OPEN MANIPULATOR JOINT  -->
+    <joint name="base_to_link1" type="fixed">
+      <origin xyz="-0.092 0.0 0.091" rpy="0 0 0"/>
+      <parent link="base_link"/>
+      <child link="link1"/>
+    </joint>
+  </xacro:if>
 </robot>
