Commit message: xacro additions for terrain + low light

File: turtlebot3_manipulation_gazebo/urdf/turtlebot3_pi_base.xacro (robot description, xacro)
@@ -4,4 +4,6 @@
   <!--  if gazebo=True, enable SDF specific tags  -->
   <xacro:arg name="gazebo" default="True"/>
+  <xacro:arg name="offroad_turtlebot" default="False"/>
+  <xacro:property name="sf" value="2.0"/>
   <!--  Begin Model Description  -->
   <link name="base_footprint"/>
@@ -33,157 +35,285 @@
     <origin xyz="0 0 0.010" rpy="0 0 0"/>
   </joint>
-  <link name="wheel_left_link">
-    <visual>
-      <origin xyz="0 0 0" rpy="1.57 0 0"/>
-      <geometry>
-        <mesh filename="file://$(find turtlebot3_description)/meshes/wheels/left_tire.stl" scale="0.001 0.001 0.001"/>
-      </geometry>
-      <material name="dark"/>
-    </visual>
-    <collision>
-      <origin xyz="0 0 0" rpy="0 0 0"/>
-      <geometry>
-        <cylinder length="0.018" radius="0.033"/>
-        <!-- Probably not supported by URDF... Will OMIT FOR NOW. TODO- REVISIT -->
-<!--        <xacro:if value="$(arg gazebo)">-->
-<!--          <surface>-->
-            <!-- This friction pamareter don't contain reliable data!! -->
-            <!--
-            <friction>
-              <ode>
-                <mu>100000.0</mu>
-                <mu2>100000.0</mu2>
-                <fdir1>0 0 0</fdir1>
-                <slip1>0.0</slip1>
-                <slip2>0.0</slip2>
-              </ode>
-            </friction>
-            <contact>
-              <ode>
-                <soft_cfm>0</soft_cfm>
-                <soft_erp>0.2</soft_erp>
-                <kp>1e+5</kp>
-                <kd>1</kd>
-                <max_vel>0.01</max_vel>
-                <min_depth>0.001</min_depth>
-              </ode>
-            </contact>
-          </surface>
-        </xacro:if> -->
-      </geometry>
-    </collision>
-    <inertial>
-      <origin xyz="0 0 0" />
-      <mass value="2.8498940e-02" />
-      <inertia ixx="1.1175580e-05" ixy="-4.2369783e-11" ixz="-5.9381719e-09"
-               iyy="1.1192413e-05" iyz="-1.4400107e-11"
-               izz="2.0712558e-05" />
+<!--        TODO: SCALE WHEELS TO MAKE THEM "ALL TERRAIN" -->
+  <xacro:if value="$(arg offroad_turtlebot)">
+    <link name="wheel_left_link">
+      <visual>
+        <origin xyz="0 0 0" rpy="1.57 0 0"/>
+        <geometry>
+          <mesh filename="file://$(find turtlebot3_description)/meshes/wheels/left_tire.stl" scale="${0.001 * sf} ${0.001 * sf} ${0.001 * sf}"/>
+        </geometry>
+        <material name="dark"/>
+      </visual>
+      <collision>
+        <origin xyz="0 0 0" rpy="0 0 0"/>
+        <geometry>
+          <cylinder length="${0.018 * sf}" radius="${sf * 0.033}"/>
+        </geometry>
+      </collision>
+      <inertial>
+        <origin xyz="0 0 0" />
+        <mass value="${sf**3 * 2.8498940e-02}" />
+        <inertia ixx="${sf**3 * 1.1175580e-05}" ixy="${sf**3 * -4.2369783e-11}" ixz="${sf**3 * -5.9381719e-09}"
+                 iyy="${sf**3 * 1.1192413e-05}" iyz="${sf**3 * -1.4400107e-11}"
+                 izz="${sf**3 * 2.0712558e-05}" />
+        </inertial>
+    </link>
+    <joint name="wheel_left_joint" type="continuous">
+      <parent link="base_link"/>
+      <child link="wheel_left_link"/>
+      <origin xyz="0.0 0.144 0.023" rpy="-1.57 0 0"/>
+      <axis xyz="0 0 1"/>
+      <xacro:if value="$(arg gazebo)">
+        <dynamics damping="0.2" friction="0.5"/>
+      </xacro:if>
+    </joint>
+    <link name="wheel_right_link">
+      <visual>
+        <origin xyz="0 0 0" rpy="1.57 0 0"/>
+        <geometry>
+          <mesh filename="file://$(find turtlebot3_description)/meshes/wheels/left_tire.stl" scale="${0.001 * sf} ${0.001 * sf} ${0.001 * sf}"/>
+        </geometry>
+        <material name="dark"/>
+      </visual>
+      <collision>
+        <origin xyz="0 0 0" rpy="0 0 0"/>
+        <geometry>
+          <cylinder length="${0.018 * sf}" radius="${sf * 0.033}"/>
+        </geometry>
+      </collision>
+      <inertial>
+        <origin xyz="0 0 0" />
+        <mass value="${sf**3 * 2.8498940e-02}" />
+        <inertia ixx="${sf**3 * 1.1175580e-05}" ixy="${sf**3 * -4.2369783e-11}" ixz="${sf**3 * -5.9381719e-09}"
+                 iyy="${sf**3 * 1.1192413e-05}" iyz="${sf**3 * -1.4400107e-11}"
+                 izz="${sf**3 * 2.0712558e-05}" />
+        </inertial>
+    </link>
+    <joint name="wheel_right_joint" type="continuous">
+      <parent link="base_link"/>
+      <child link="wheel_right_link"/>
+      <origin xyz="0.0 -0.144 0.023" rpy="-1.57 0 0"/>
+      <axis xyz="0 0 1"/>
+      <xacro:if value="$(arg gazebo)">
+        <dynamics damping="0.2" friction="0.5"/>
+      </xacro:if>
+    </joint>
+    <link name="caster_back_right_link">
+      <visual>
+        <origin xyz="0 0 0" rpy="0 0 0"/>
+        <geometry>
+          <sphere radius="${0.033 * sf - 0.028}"/>
+        </geometry>
+      </visual>
+      <collision>
+        <origin xyz="0 0 0" rpy="0 0 0"/>
+        <geometry>
+          <sphere radius="${0.033 * sf - 0.028}"/>
+        </geometry>
+      </collision>
+      <inertial>
+        <origin xyz="0 0 0" />
+        <mass value="${sf**3 * 0.005}" />
+        <inertia ixx="${sf**3 * 0.001}" ixy="${sf**3 * 0.0}" ixz="${sf**3 * 0.0}"
+                 iyy="${sf**3 * 0.001}" iyz="${sf**3 * 0.0}"
+                 izz="${sf**3 * 0.001}" />
       </inertial>
-  </link>
-  <joint name="wheel_left_joint" type="continuous">
-    <parent link="base_link"/>
-    <child link="wheel_left_link"/>
-    <origin xyz="0.0 0.144 0.023" rpy="-1.57 0 0"/>
-    <axis xyz="0 0 1"/>
+    </link>
     <xacro:if value="$(arg gazebo)">
-      <dynamics damping="0.2" friction="0.5"/>
-    </xacro:if>
-  </joint>
-  <link name="wheel_right_link">
-    <visual>
-      <origin xyz="0 0 0" rpy="1.57 0 0"/>
-      <geometry>
-        <mesh filename="file://$(find turtlebot3_description)/meshes/wheels/right_tire.stl" scale="0.001 0.001 0.001"/>
-      </geometry>
-      <material name="dark"/>
-    </visual>
-    <collision>
-      <origin xyz="0 0 0" rpy="0 0 0"/>
-      <geometry>
-        <cylinder length="0.018" radius="0.033"/>
-        <!-- Probably not supported by URDF... Will OMIT FOR NOW. TODO- REVISIT -->
-<!--        <xacro:if value="$(arg gazebo)">-->
-<!--          <surface>-->
-            <!-- This friction pamareter don't contain reliable data!! -->
-            <!--
-            <friction>
-              <ode>
-                <mu>100000.0</mu>
-                <mu2>100000.0</mu2>
-                <fdir1>0 0 0</fdir1>
-                <slip1>0.0</slip1>
-                <slip2>0.0</slip2>
-              </ode>
-            </friction>
-            <contact>
-              <ode>
-                <soft_cfm>0</soft_cfm>
-                <soft_erp>0.2</soft_erp>
-                <kp>1e+5</kp>
-                <kd>1</kd>
-                <max_vel>0.01</max_vel>
-                <min_depth>0.001</min_depth>
-              </ode>
-            </contact>
-          </surface>
-        </xacro:if> -->
-      </geometry>
-    </collision>
-    <inertial>
-      <origin xyz="0 0 0" />
-      <mass value="2.8498940e-02" />
-      <inertia ixx="1.1175580e-05" ixy="-4.2369783e-11" ixz="-5.9381719e-09"
-               iyy="1.1192413e-05" iyz="-1.4400107e-11"
-               izz="2.0712558e-05" />
+      <!-- Represent ball joint by 2 additional links and joints   -->
+      <link name="caster_back_right_link_proxy1">
+        <inertial>
+          <origin xyz="0 0 0" />
+          <mass value="0.005" />
+          <inertia ixx="0.001" ixy="0.0" ixz="0.0"
+                   iyy="0.001" iyz="0.0"
+                   izz="0.001" />
+        </inertial>
+      </link>
+      <link name="caster_back_right_link_proxy2">
+        <inertial>
+          <origin xyz="0 0 0" />
+          <mass value="0.005" />
+          <inertia ixx="0.001" ixy="0.0" ixz="0.0"
+                   iyy="0.001" iyz="0.0"
+                   izz="0.001" />
+        </inertial>
+      </link>
+      <joint name="caster_back_right_joint_x" type="continuous">
+        <parent link="base_link"/>
+        <child link="caster_back_right_link_proxy1"/>
+        <origin xyz="-0.177 -0.064 -0.005" rpy="-1.57 0 0"/>
+        <axis xyz="1 0 0"/>
+        <dynamics damping="0.1" friction="0.2"/>
+      </joint>
+      <joint name="caster_back_right_joint_y" type="continuous">
+        <parent link="caster_back_right_link_proxy1"/>
+        <child link="caster_back_right_link_proxy2"/>
+        <origin xyz="0 0 0" rpy="0 0 0"/>
+        <axis xyz="0 1 0"/>
+        <dynamics damping="0.1" friction="0.2"/>
+      </joint>
+      <joint name="caster_back_right_joint_z" type="continuous">
+        <parent link="caster_back_right_link_proxy2"/>
+        <child link="caster_back_right_link"/>
+        <origin xyz="0 0 0" rpy="0 0 0"/>
+        <axis xyz="0 0 1"/>
+       <dynamics damping="0.1" friction="0.2"/>
+      </joint>
+    </xacro:if>
+    <xacro:if value="${not $(arg gazebo)}">
+      <joint name="caster_back_right_joint" type="fixed">
+        <parent link="base_link"/>
+        <child link="caster_back_right_link"/>
+        <origin xyz="-0.177 -0.064 -0.004" rpy="-1.57 0 0"/>
+      </joint>
+    </xacro:if>
+    <link name="caster_back_left_link">
+      <visual>
+        <origin xyz="0 0 0" rpy="0 0 0"/>
+        <geometry>
+          <sphere radius="${0.033 * sf - 0.028}"/>
+        </geometry>
+      </visual>
+      <collision>
+        <origin xyz="0 0 0" rpy="0 0 0"/>
+        <geometry>
+          <sphere radius="${0.033 * sf - 0.028}"/>
+        </geometry>
+      </collision>
+      <inertial>
+        <origin xyz="0 0 0" />
+        <mass value="${sf**3 * 0.005}" />
+        <inertia ixx="${sf**3 * 0.001}" ixy="${sf**3 * 0.0}" ixz="${sf**3 * 0.0}"
+                 iyy="${sf**3 * 0.001}" iyz="${sf**3 * 0.0}"
+                 izz="${sf**3 * 0.001}" />
       </inertial>
-  </link>
-  <joint name="wheel_right_joint" type="continuous">
-    <parent link="base_link"/>
-    <child link="wheel_right_link"/>
-    <origin xyz="0.0 -0.144 0.023" rpy="-1.57 0 0"/>
-    <axis xyz="0 0 1"/>
+    </link>
     <xacro:if value="$(arg gazebo)">
-      <dynamics damping="0.2" friction="0.5"/>
-    </xacro:if>
-  </joint>
-  <link name="caster_back_right_link">
-    <visual>
-      <origin xyz="0 0 0" rpy="0 0 0"/>
-      <geometry>
-        <sphere radius="0.005"/>
-      </geometry>
-    </visual>
-    <collision>
-      <origin xyz="0 0 0" rpy="0 0 0"/>
-      <geometry>
-        <sphere radius="0.005"/>
-        <!--
-        TODO- Consider adding to gazebo version
-        <surface>
-          <contact>
-            <ode>
-              <soft_cfm>0</soft_cfm>
-              <soft_erp>0.2</soft_erp>
-              <kp>1e+5</kp>
-              <kd>1</kd>
-              <max_vel>0.01</max_vel>
-              <min_depth>0.001</min_depth>
-            </ode>
-          </contact>
-        </surface>
-        -->
-      </geometry>
-    </collision>
-    <inertial>
-      <origin xyz="0 0 0" />
-      <mass value="0.005" />
-      <inertia ixx="0.001" ixy="0.0" ixz="0.0"
-               iyy="0.001" iyz="0.0"
-               izz="0.001" />
-    </inertial>
-  </link>
-  <xacro:if value="$(arg gazebo)">
-    <!-- Represent ball joint by 2 additional links and joints   -->
-    <link name="caster_back_right_link_proxy1">
+      <!-- Represent ball joint by 2 additional links and joints   -->
+      <link name="caster_back_left_link_proxy1">
+        <inertial>
+          <origin xyz="0 0 0" />
+          <mass value="0.005" />
+          <inertia ixx="0.001" ixy="0.0" ixz="0.0"
+                   iyy="0.001" iyz="0.0"
+                   izz="0.001" />
+        </inertial>
+      </link>
+      <link name="caster_back_left_link_proxy2">
+        <inertial>
+          <origin xyz="0 0 0" />
+          <mass value="0.005" />
+          <inertia ixx="0.001" ixy="0.0" ixz="0.0"
+                   iyy="0.001" iyz="0.0"
+                   izz="0.001" />
+        </inertial>
+      </link>
+      <joint name="caster_back_left_joint_x" type="continuous">
+        <parent link="base_link"/>
+        <child link="caster_back_left_link_proxy1"/>
+        <origin xyz="-0.177 0.064 -0.005" rpy="-1.57 0 0"/>
+        <axis xyz="1 0 0"/>
+        <dynamics damping="0.1" friction="0.2"/>
+      </joint>
+      <joint name="caster_back_left_joint_y" type="continuous">
+        <parent link="caster_back_left_link_proxy1"/>
+        <child link="caster_back_left_link_proxy2"/>
+        <origin xyz="0 0 0" rpy="0 0 0"/>
+        <axis xyz="0 1 0"/>
+        <dynamics damping="0.1" friction="0.2"/>
+      </joint>
+      <joint name="caster_back_left_joint_z" type="continuous">
+        <parent link="caster_back_left_link_proxy2"/>
+        <child link="caster_back_left_link"/>
+        <origin xyz="0 0 0" rpy="0 0 0"/>
+        <axis xyz="0 0 1"/>
+        <dynamics damping="0.1" friction="0.2"/>
+      </joint>
+    </xacro:if>
+    <xacro:if value="${not $(arg gazebo)}">
+      <joint name="caster_back_left_joint" type="fixed">
+        <parent link="base_link"/>
+        <child link="caster_back_left_link"/>
+        <origin xyz="-0.177 0.064 -0.004" rpy="-1.57 0 0"/>
+      </joint>
+    </xacro:if>
+  </xacro:if>
+  <xacro:if value="${not $(arg offroad_turtlebot)}">
+    <link name="wheel_left_link">
+      <visual>
+        <origin xyz="0 0 0" rpy="1.57 0 0"/>
+        <geometry>
+          <mesh filename="file://$(find turtlebot3_description)/meshes/wheels/left_tire.stl" scale="0.001 0.001 0.001"/>
+        </geometry>
+        <material name="dark"/>
+      </visual>
+      <collision>
+        <origin xyz="0 0 0" rpy="0 0 0"/>
+        <geometry>
+          <cylinder length="0.018" radius="0.033"/>
+        </geometry>
+      </collision>
+      <inertial>
+        <origin xyz="0 0 0" />
+        <mass value="2.8498940e-02" />
+        <inertia ixx="1.1175580e-05" ixy="-4.2369783e-11" ixz="-5.9381719e-09"
+                 iyy="1.1192413e-05" iyz="-1.4400107e-11"
+                 izz="2.0712558e-05" />
+        </inertial>
+    </link>
+    <joint name="wheel_left_joint" type="continuous">
+      <parent link="base_link"/>
+      <child link="wheel_left_link"/>
+      <origin xyz="0.0 0.144 0.023" rpy="-1.57 0 0"/>
+      <axis xyz="0 0 1"/>
+      <xacro:if value="$(arg gazebo)">
+        <dynamics damping="0.2" friction="0.5"/>
+      </xacro:if>
+    </joint>
+    <link name="wheel_right_link">
+      <visual>
+        <origin xyz="0 0 0" rpy="1.57 0 0"/>
+        <geometry>
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
File: turtlebot3_manipulation_gazebo/urdf/turtlebot3_pi_gazebo.xacro (robot description, xacro)
@@ -4,4 +4,7 @@
   <!--  if gazebo=True, enable SDF specific tags  -->
   <xacro:arg name="gazebo" default="True"/>
+  <xacro:arg name="offroad_turtlebot" default="False"/>
+  <xacro:arg name="flashlight" default="False"/>
+  <xacro:property name="sf" value="2.0"/>
   <xacro:if value="$(arg gazebo)">
     <gazebo reference="base_link">
@@ -174,9 +177,18 @@
         <right_joint>wheel_right_joint</right_joint>
         <!-- kinematics -->
-        <wheel_separation>0.287</wheel_separation>
-        <wheel_diameter>0.066</wheel_diameter>
-        <!-- limits -->
-        <max_wheel_torque>20</max_wheel_torque>
-        <max_wheel_acceleration>1.0</max_wheel_acceleration>
+        <xacro:if value="$(arg offroad_turtlebot)">
+          <wheel_separation>0.287</wheel_separation>
+          <wheel_diameter>${sf*0.066}</wheel_diameter>
+          <!-- limits -->
+          <max_wheel_torque>${sf*20}</max_wheel_torque>
+          <max_wheel_acceleration>1.0</max_wheel_acceleration>
+        </xacro:if>
+        <xacro:if value="${not $(arg offroad_turtlebot)}">
+          <wheel_separation>0.287</wheel_separation>
+          <wheel_diameter>0.066</wheel_diameter>
+          <!-- limits -->
+          <max_wheel_torque>20</max_wheel_torque>
+          <max_wheel_acceleration>1.0</max_wheel_acceleration>
+        </xacro:if>
         <command_topic>cmd_vel</command_topic>
         <!-- output -->
@@ -200,4 +212,79 @@
       </plugin>
     </gazebo>
+    <xacro:if value="$(arg flashlight)">
+      <!--    create links to attack flashlights to-->
+      <link name="flashlight_1"/>
+      <link name="flashlight_2"/>
+      <joint name="flashlight_joint_1" type="fixed">
+        <parent link="base_link"/>
+        <child link="flashlight_1"/>
+        <origin rpy="0.0 0.0 0.0" xyz="0.0 0.0 0.0"/>
+      </joint>
+      <joint name="flashlight_joint_2" type="fixed">
+        <parent link="base_link"/>
+        <child link="flashlight_2"/>
+        <origin rpy="0.0 0.0 0.0" xyz="0.0 0.0 0.0"/>
+      </joint>
+      <gazebo reference="flashlight_1">
+        <light name="light_1" type="spot">
+          <cast_shadows>1</cast_shadows>
+          <intensity>1</intensity>
+          <diffuse>1 1 1 1</diffuse>
+          <specular>.5 .5 .5 1 </specular>
+          <attenuation>
+            <range>20</range>
+            <linear>1</linear>
+            <constant>1</constant>
+            <quadratic>0</quadratic>
+          </attenuation>
+          <direction>0 0 -1</direction>
+          <spot>
+            <inner_angle>0.8</inner_angle>
+            <outer_angle>0.8</outer_angle>
+            <falloff>1</falloff>
+          </spot>
+          <pose>0 -0.1 0.125 0 -1.5 -0.2</pose>
+        </light>
+        <plugin name='light_control' filename='libFlashLightPlugin.so'>
+          <enable>true</enable>
+          <light>
+            <id>flashlight_1/light_1</id>
+            <color>1 1 1</color>
+            <duration>1</duration>
+            <interval>0.5</interval>
+          </light>
+        </plugin>
+      </gazebo>
+      <gazebo reference="flashlight_2">
+        <light name="light_2" type="spot">
+          <cast_shadows>1</cast_shadows>
+          <intensity>1</intensity>
+          <diffuse>1 1 1 1</diffuse>
+          <specular>.5 .5 .5 1 </specular>
+          <attenuation>
+            <range>20</range>
+            <linear>1</linear>
+            <constant>1</constant>
+            <quadratic>0</quadratic>
+          </attenuation>
+          <direction>0 0 -1</direction>
+          <spot>
+            <inner_angle>0.8</inner_angle>
+            <outer_angle>0.8</outer_angle>
+            <falloff>1</falloff>
+          </spot>
+          <pose>0 0.1 0.125 0.0 -1.5 0.2</pose>
+        </light>
+        <plugin name='light_control' filename='libFlashLightPlugin.so'>
+          <enable>true</enable>
+          <light>
+            <id>flashlight_2/light_2</id>
+            <color>1 1 1</color>
+            <duration>1</duration>
+            <interval>0.5</interval>
+          </light>
+        </plugin>
+      </gazebo>
+    </xacro:if>
   </xacro:if>
 </robot>

File: turtlebot3_manipulation_gazebo/urdf/turtlebot3_pi_manipulator.xacro (robot description, xacro)
@@ -1,4 +1,6 @@
 <?xml version="1.0" ?>
 <robot name="turtlebot3_manipulator" xmlns:xacro="http://ros.org/wiki/xacro">
+  <!-- For "terrain" simulations environments -->
+  <xacro:arg name="offroad_turtlebot" default="False"/>
   <!-- Import Rviz colors -->
   <xacro:include filename="$(find open_manipulator_x_description)/urdf/materials.xacro" />
