Commit message: updating xacro for open_manipulator hardware control

File: turtlebot3_manipulation_gazebo/urdf/turtlebot3_pi.xacro (robot description, xacro)
@@ -3,4 +3,7 @@
 <robot name="turtlebot3_manipulation" xmlns:xacro="http://ros.org/wiki/xacro">
   <xacro:arg name="gazebo" default="True"/>
+  <xacro:arg name="offroad_turtlebot" default="False"/>
+  <xacro:arg name="scale_factor" default="1.0"/>
+  <xacro:property name="sf" value="$(arg scale_factor)"/>
   <!--  TURTLEBOT3 WAFFLE PI  -->
   <xacro:include filename="$(find turtlebot3_manipulation_gazebo)/urdf/turtlebot3_pi_base.xacro"/>

File: turtlebot3_manipulation_gazebo/urdf/turtlebot3_pi_base.xacro (robot description, xacro)
@@ -5,5 +5,6 @@
   <xacro:arg name="gazebo" default="True"/>
   <xacro:arg name="offroad_turtlebot" default="False"/>
-  <xacro:property name="sf" value="2.0"/>
+  <xacro:arg name="scale_factor" default="1.0"/>
+  <xacro:property name="sf" value="$(arg scale_factor)"/>
   <!--  Begin Model Description  -->
   <link name="base_footprint"/>
@@ -35,5 +36,4 @@
     <origin xyz="0 0 0.010" rpy="0 0 0"/>
   </joint>
-<!--        TODO: SCALE WHEELS TO MAKE THEM "ALL TERRAIN" -->
   <xacro:if value="$(arg offroad_turtlebot)">
     <link name="wheel_left_link">

File: turtlebot3_manipulation_gazebo/urdf/turtlebot3_pi_gazebo.xacro (robot description, xacro)
@@ -5,6 +5,7 @@
   <xacro:arg name="gazebo" default="True"/>
   <xacro:arg name="offroad_turtlebot" default="False"/>
+  <xacro:arg name="scale_factor" default="1.0"/>
+  <xacro:property name="sf" value="$(arg scale_factor)"/>
   <xacro:arg name="flashlight" default="False"/>
-  <xacro:property name="sf" value="2.0"/>
   <xacro:if value="$(arg gazebo)">
     <gazebo reference="base_link">
@@ -228,4 +229,5 @@
       <gazebo reference="flashlight_1">
         <light name="light_1" type="spot">
+          <visualize>0</visualize>
           <cast_shadows>1</cast_shadows>
           <intensity>1</intensity>
@@ -258,4 +260,5 @@
       <gazebo reference="flashlight_2">
         <light name="light_2" type="spot">
+          <visualize>0</visualize>
           <cast_shadows>1</cast_shadows>
           <intensity>1</intensity>

File: turtlebot3_manipulation_gazebo/urdf/turtlebot3_pi_manipulator.xacro (robot description, xacro)
@@ -14,4 +14,5 @@
     <xacro:include filename="$(find open_manipulator_x_description)/urdf/open_manipulator_x.transmission.xacro"/>
     <xacro:include filename="$(find open_manipulator_x_description)/urdf/open_manipulator_x.gazebo.xacro"/>
+    <xacro:include filename="$(find open_manipulator_x_description)/urdf/open_manipulator_x.controller.xacro"/>
     <!-- TURTLEBOT-OPEN MANIPULATOR JOINT  -->
     <joint name="base_to_link1" type="fixed">
