Commit message: launch tweaks and new env

File: turtlebot3_manipulation_gazebo/urdf/turtlebot3_pi_gazebo.xacro (robot description, xacro)
@@ -36,9 +36,15 @@
       <maxVel>10.0</maxVel>
     </gazebo>
+    <gazebo reference="caster_back_left_link">
+      <material>Gazebo/FlatBlack</material>
+    </gazebo>
+    <gazebo reference="caster_back_right_link">
+      <material>Gazebo/FlatBlack</material>
+    </gazebo>
     <gazebo reference="base_scan">
       <material>Gazebo/FlatBlack</material>
       <sensor name="hls_lfcd_lds" type="ray">
         <always_on>true</always_on>
-        <visualize>true</visualize>
+        <visualize>false</visualize>
         <pose>0 0 0 0 0 0</pose>
 <!--        <pose>-1.064 0 0.121 0 0 0</pose>-->
@@ -80,5 +86,5 @@
       <sensor name="camera" type="camera">
         <always_on>true</always_on>
-        <visualize>true</visualize>
+        <visualize>false</visualize>
         <update_rate>30</update_rate>
         <camera name="picam">
@@ -229,5 +235,4 @@
       <gazebo reference="flashlight_1">
         <light name="light_1" type="spot">
-          <visualize>0</visualize>
           <cast_shadows>1</cast_shadows>
           <intensity>1</intensity>
@@ -235,5 +240,5 @@
           <specular>.5 .5 .5 1 </specular>
           <attenuation>
-            <range>20</range>
+            <range>40</range>
             <linear>1</linear>
             <constant>1</constant>
@@ -260,5 +265,4 @@
       <gazebo reference="flashlight_2">
         <light name="light_2" type="spot">
-          <visualize>0</visualize>
           <cast_shadows>1</cast_shadows>
           <intensity>1</intensity>
@@ -266,5 +270,5 @@
           <specular>.5 .5 .5 1 </specular>
           <attenuation>
-            <range>20</range>
+            <range>40</range>
             <linear>1</linear>
             <constant>1</constant>
